File: sch/rvisitor_module_board_v1/rvisitor_module_board_v1/power.kicad_sch (KiCad schematic)
At the start: 0 parts

Commit message: [sch] rvisitor_module_board_v1 => power lines added
Parts:
- added J19, J20, J21: 39290043, 39290043:MOLEX_39290043, symbol MiniFit:39290043
Connections:
- new net +3.3V: J19.1, J19.2
- new net +5V: J20.1, J20.2
- new net GNDREF: J19.3, J19.4, J20.3, J20.4, J21.3, J21.4
- new net Vdrive: J21.1, J21.2
