File: sch/maket/maket.kicad_pcb (KiCad board)
At the start: 2 copper layers, 0 parts

Commit message: maket pcb start. maket add footprints. module_board_v1 start
Parts:
- added D1: 1N5820, Diode_THT:D_DO-201AD_P15.24mm_Horizontal, F.Cu at (155.9, 197.1)
- added D2: 1N5820, Diode_THT:D_DO-201AD_P15.24mm_Horizontal, F.Cu at (155.9, 203.9)
- added D3: 1N5820, Diode_THT:D_DO-201AD_P15.24mm_Horizontal, F.Cu at (155.9, 210.6)
- added D4: 1N5820, Diode_THT:D_DO-201AD_P15.24mm_Horizontal, F.Cu at (155.9, 217.4)
- added DD1: ~, CH32V307VCT6_dev_board:CH32V307VCT6 dev board, F.Cu at (145.1, 71.3)
- added DD2: ~, L9110S:L9110S, F.Cu at (61.3, 96.7)
- added DD3: ~, L9110S:L9110S, F.Cu at (234.0, 87.8)
- added DD4: ~, CD74HC4067_good:CD74HC4067_GOOD, F.Cu at (102.5, 85.5)
- added DD5: ~, CD74HC4067_good:CD74HC4067_GOOD, F.Cu at (201.0, 85.2)
- added DD6: ~, INA226:INA226, F.Cu at (161.7, 180.5)
- added J1: YL-63, Connector_PinHeader_2.54mm:PinHeader_1x03_P2.54mm_Vertical, F.Cu at (256.9, 26.8)
- added J10: HC-SR04, Connector_PinHeader_2.54mm:PinHeader_1x04_P2.54mm_Vertical, F.Cu at (104.2, 172.5)
- added J11: HC-SR04, Connector_PinHeader_2.54mm:PinHeader_1x04_P2.54mm_Vertical, F.Cu at (108.8, 172.5)
- added J12: HC-SR04, Connector_PinHeader_2.54mm:PinHeader_1x04_P2.54mm_Vertical, F.Cu at (113.5, 172.5)
- added J13: UART_CMD_IFACE, Connector_PinHeader_2.54mm:PinHeader_1x04_P2.54mm_Vertical, F.Cu at (274.7, 87.8)
- added J14: Encoder4, Connector_JST:JST_PH_S4B-PH-K_1x04_P2.00mm_Horizontal, F.Cu at (165.6, 130.0)
- added J15: Encoder3, Connector_JST:JST_PH_S4B-PH-K_1x04_P2.00mm_Horizontal, F.Cu at (165.6, 139.6)
- added J16: Encoder2, Connector_JST:JST_PH_S4B-PH-K_1x04_P2.00mm_Horizontal, F.Cu at (165.6, 149.3)
- added J17: Encoder1, Connector_JST:JST_PH_S4B-PH-K_1x04_P2.00mm_Horizontal, F.Cu at (165.6, 158.9)
- added J2: YL-63, Connector_PinHeader_2.54mm:PinHeader_1x03_P2.54mm_Vertical, F.Cu at (43.5, 26.8)
- added J3: YL-63, Connector_PinHeader_2.54mm:PinHeader_1x03_P2.54mm_Vertical, F.Cu at (48.6, 153.8)
- added J4: YL-63, Connector_PinHeader_2.54mm:PinHeader_1x03_P2.54mm_Vertical, F.Cu at (256.9, 153.8)
- added J5: DC_Conn, Connector_JST:JST_PH_S2B-PH-K_1x02_P2.00mm_Horizontal, F.Cu at (264.5, 85.8)
- added J6: DC_Conn, Connector_JST:JST_PH_S2B-PH-K_1x02_P2.00mm_Horizontal, F.Cu at (264.5, 96.0)
- added J7: DC_Conn, Connector_JST:JST_PH_S2B-PH-K_1x02_P2.00mm_Horizontal, F.Cu at (33.4, 100.0)
- added J8: DC_Conn, Connector_JST:JST_PH_S2B-PH-K_1x02_P2.00mm_Horizontal, F.Cu at (33.4, 87.2)
- added J9: HC-SR04, Connector_PinHeader_2.54mm:PinHeader_1x04_P2.54mm_Vertical, F.Cu at (99.5, 172.5)

Commit message: PCB module. readme update
Parts:
- J10, J11, J12, J13, J9: footprint Connector_PinHeader_2.54mm:PinHeader_1x04_P2.54mm_Vertical -> Connector_PinSocket_2.54mm:PinSocket_1x04_P2.54mm_Vertical
- moved J12 163.5 mm to (249.3, 81.5)
- moved D2 162.5 mm to (170.5, 42.1), turned to 180 degrees
- moved J10 146.4 mm to (145.1, 31.9), turned to 90 degrees
- moved D4 130.5 mm to (218.8, 103.0)
- moved D1 121.4 mm to (79.1, 103.0), turned to 180 degrees
- moved J13 115.7 mm to (165.5, 125.9), turned to -90 degrees
- moved J17 114.7 mm to (117.7, 54.7), turned to 180 degrees
- moved J16 97.4 mm to (188.8, 54.7), turned to 180 degrees
- moved J9 96.5 mm to (51.2, 89.0), turned to 180 degrees
- moved D3 78.1 mm to (168.0, 133.5), turned to -90 degrees
- moved DD6 54.5 mm to (136.2, 132.2)
- moved J15 53.3 mm to (116.7, 118.4)
- moved J1 44.4 mm to (218.8, 49.7)
- moved J4 44.4 mm to (218.8, 131.0)
- moved J11 42.0 mm to (145.1, 151.3), turned to 90 degrees
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Connections:
- D2 pad 2: GNDD -> Net-(D2-A)
- J10 pad 3: GNDD -> Net-(D2-A)
