File: sch/maket/maket.kicad_sch (KiCad schematic)
At the start: 29 parts, among them J1 YL-63, J10 HC-SR04, J11 HC-SR04, J12 HC-SR04, J13 UART_CMD_IFACE, J14 Encoder4, J15 Encoder3, J16 Encoder2, J17 Encoder1, J2 YL-63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

Commit message: maket pcb start. maket add footprints. module_board_v1 start
Parts:
- removed R3: 100R, symbol Device:R_Small
- removed R4: 200R, symbol Device:R_Small
- DD1: footprint (none) -> CH32V307VCT6_dev_board:CH32V307VCT6 dev board
- DD2, DD3: footprint (none) -> L9110S:L9110S
- DD4, DD5: footprint (none) -> CD74HC4067_good:CD74HC4067_GOOD
- DD6: footprint (none) -> INA226:INA226
- J1, J2, J3, J4: footprint (none) -> Connector_PinHeader_2.54mm:PinHeader_1x03_P2.54mm_Vertical
- J10, J11, J12, J13, J9: footprint (none) -> Connector_PinHeader_2.54mm:PinHeader_1x04_P2.54mm_Vertical
- J14, J15, J16, J17: footprint (none) -> Connector_JST:JST_PH_S4B-PH-K_1x04_P2.00mm_Horizontal
- J5, J6, J7, J8: footprint (none) -> Connector_JST:JST_PH_S2B-PH-K_1x02_P2.00mm_Horizontal
Connections:
- net +3.3V: no longer DD6.0 (IN+), DD6.1 (IN-)
- net GNDD: now also D2.2 (A), DD6.3 (ALE), J10.3 (Echo); no longer DD1.3 (GND)
- net HCSR_ECHO: now also D1.1 (K), D2.1 (K), D3.1 (K), D4.1 (K)
Other:
- moved on the sheet: D1, D2, D3, D4, DD5, J10, J11, J12, J9

Commit message: PCB module. readme update
Parts:
- J10, J11, J12, J13, J9: footprint Connector_PinHeader_2.54mm:PinHeader_1x04_P2.54mm_Vertical -> Connector_PinSocket_2.54mm:PinSocket_1x04_P2.54mm_Vertical
Connections:
- net GNDD: no longer D2.2 (A), J10.3 (Echo)
- new net: D2.2 (A), J10.3 (Echo)
Changed lines of the file:
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@@
 	)
 	(junction
-		(at 326.39 115.57)
-		(diameter 0)
-		(color 0 0 0 0)
-	)
-	(junction
 		(at 231.14 43.18)
 		(diameter 0)
@@
 	(wire
 		(pts
+			(xy 322.58 115.57) (xy 328.93 115.57)
+		)
+		(stroke
+			(width 0)
+			(type default)
+		)
+	)
+	(wire
+		(pts
 			(xy 280.67 229.87) (xy 280.67 246.38)
 		)
@@
 	(wire
 		(pts
-			(xy 326.39 115.57) (xy 326.39 118.11)
+			(xy 326.39 100.33) (xy 326.39 118.11)
 		)
 		(stroke
@@
 	(wire
 		(pts
-			(xy 322.58 115.57) (xy 326.39 115.57)
-		)
-		(stroke
-			(width 0)
-			(type default)
-		)
-	)
-	(wire
-		(pts
 			(xy 252.73 199.39) (xy 285.75 199.39)
 		)
@@
 	(wire
 		(pts
-			(xy 326.39 115.57) (xy 328.93 115.57)
-		)
-		(stroke
-			(width 0)
-			(type default)
-		)
-	)
-	(wire
-		(pts
 			(xy 295.91 100.33) (xy 302.26 100.33)
 		)
@@
 	(wire
 		(pts
-			(xy 326.39 100.33) (xy 326.39 115.57)
-		)
-		(stroke
-			(width 0)
-			(type default)
-		)
-	)
-	(wire
-		(pts
 			(xy 292.1 36.83) (xy 320.04 36.83)
 		)
@@
 			)
 		)
-		(property "Footprint" "Connector_PinHeader_2.54mm:PinHeader_1x04_P2.54mm_Vertical"
+		(property "Footprint" "Connector_PinSocket_2.54mm:PinSocket_1x04_P2.54mm_Vertical"
 			(at 334.01 95.25 0)
 			(effects
@@
 			)
 		)
-		(property "Footprint" "Connector_PinHeader_2.54mm:PinHeader_1x04_P2.54mm_Vertical"
+		(property "Footprint" "Connector_PinSocket_2.54mm:PinSocket_1x04_P2.54mm_Vertical"
 			(at 334.01 113.03 0)
 			(effects
@@
 			)
 		)
-		(property "Footprint" "Connector_PinHeader_2.54mm:PinHeader_1x04_P2.54mm_Vertical"
+		(property "Footprint" "Connector_PinSocket_2.54mm:PinSocket_1x04_P2.54mm_Vertical"
 			(at 332.74 128.27 0)
 			(effects
@@
 			)
 		)
-		(property "Footprint" "Connector_PinHeader_2.54mm:PinHeader_1x04_P2.54mm_Vertical"
+		(property "Footprint" "Connector_PinSocket_2.54mm:PinSocket_1x04_P2.54mm_Vertical"
 			(at 332.74 143.51 0)
 			(effects
@@
 			)
 		)
-		(property "Footprint" "Connector_PinHeader_2.54mm:PinHeader_1x04_P2.54mm_Vertical"
+		(property "Footprint" "Connector_PinSocket_2.54mm:PinSocket_1x04_P2.54mm_Vertical"
 			(at 97.79 157.48 0)
 			(effects
